File: rp-2040 devboard.kicad_pcb (KiCad board)
At the start: 2 copper layers, 20.7 x 51.8 mm, 32 parts, among them J1 USB_C_Receptacle_USB2.0_16P, J2 Conn_01x20, J3 Conn_01x20, J4 Conn_01x03, SW1 SW_Push, U1 RP2040, U2 APS1604M-3SQRx-ZR, U4 MCP1700x-330xxTT, Y1 Crystal_GND24

Commit message: new BOM
Parts:
- SW1: footprint Button_Switch_SMD:SW_Push_SPST_NO_Alps_SKRK -> Button_Switch_SMD:SW_SPST_PTS810
- moved SW1 0.28 mm to (91.2, 109.5), turned to 0 degrees
Routing:
- net Net-(R6-Pad1): track 2.06 -> 5.56 mm
Changed lines of the file:
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@@
 		)
 	)
-	(footprint "Button_Switch_SMD:SW_Push_SPST_NO_Alps_SKRK"
+	(footprint "Button_Switch_SMD:SW_SPST_PTS810"
 		(layer "F.Cu")
-		(at 90.975 109.6 180)
-		(descr "http://www.alps.com/prod/info/E/HTML/Tact/SurfaceMount/SKRK/SKRKAHE020.html")
-		(tags "SMD SMT button")
+		(at 91.25 109.55)
+		(descr "C&K Components, PTS 810 Series, Microminiature SMT Top Actuated, http://www.ckswitches.com/media/1476/pts810.pdf")
+		(tags "SPST Button Switch")
 		(property "Reference" "SW1"
-			(at 0 -2.25 0)
+			(at 0 -2.6 0)
 			(layer "F.SilkS")
-			(hide yes)
 			(effects
 				(font
@@
 		)
 		(property "Value" "SW_Push"
-			(at 0 2.5 0)
+			(at 0 2.6 0)
 			(layer "F.Fab")
 			(hide yes)
@@
 		)
 		(property "Datasheet" ""
-			(at 0 0 180)
+			(at 0 0 0)
 			(unlocked yes)
 			(layer "F.Fab")
@@
 		)
 		(property "Description" ""
-			(at 0 0 180)
+			(at 0 0 0)
 			(unlocked yes)
 			(layer "F.Fab")
@@
 		(duplicate_pad_numbers_are_jumpers no)
 		(fp_line
-			(start 2.07 1.57)
-			(end -2.07 1.57)
+			(start -2.2 -1.7)
+			(end -2.2 -1.58)
 			(stroke
 				(width 0.12)
@@
 		)
 		(fp_line
-			(start 2.07 1.27)
-			(end 2.07 1.57)
+			(start -2.2 -0.57)
+			(end -2.2 0.57)
 			(stroke
 				(width 0.12)
@@
 		)
 		(fp_line
-			(start 2.07 -1.57)
-			(end 2.07 -1.27)
+			(start -2.2 1.58)
+			(end -2.2 1.7)
 			(stroke
 				(width 0.12)
@@
 		)
 		(fp_line
-			(start -2.07 1.57)
-			(end -2.07 1.27)
+			(start -2.2 1.7)
+			(end 2.2 1.7)
 			(stroke
 				(width 0.12)
@@
 		)
 		(fp_line
-			(start -2.07 -1.27)
-			(end -2.07 -1.57)
+			(start 2.2 -1.7)
+			(end -2.2 -1.7)
 			(stroke
 				(width 0.12)
@@
 		)
 		(fp_line
-			(start -2.07 -1.57)
-			(end 2.07 -1.57)
+			(start 2.2 -1.58)
+			(end 2.2 -1.7)
 			(stroke
 				(width 0.12)
@@
 		)
 		(fp_line
-			(start 2.75 1.7)
-			(end -2.75 1.7)
+			(start 2.2 0.57)
+			(end 2.2 -0.57)
+			(stroke
+				(width 0.12)
+				(type solid)
+			)
+			(layer "F.SilkS")
+		)
+		(fp_line
+			(start 2.2 1.7)
+			(end 2.2 1.58)
+			(stroke
+				(width 0.12)
+				(type solid)
+			)
+			(layer "F.SilkS")
+		)
+		(fp_line
+			(start -2.85 -1.85)
+			(end 2.85 -1.85)
 			(stroke
 				(width 0.05)
@@
 		)
 		(fp_line
-			(start 2.75 -1.7)
-			(end 2.75 1.7)
+			(start -2.85 1.85)
+			(end -2.85 -1.85)
 			(stroke
 				(width 0.05)
@@
 		)
 		(fp_line
-			(start -2.75 1.7)
-			(end -2.75 -1.7)
+			(start 2.85 -1.85)
+			(end 2.85 1.85)
 			(stroke
 				(width 0.05)
@@
 		)
 		(fp_line
-			(start -2.75 -1.7)
-			(end 2.75 -1.7)
+			(start 2.85 1.85)
+			(end -2.85 1.85)
 			(stroke
 				(width 0.05)
@@
 		)
 		(fp_line
-			(start 1.95 1.45)
-			(end -1.95 1.45)
+			(start -2.1 -1.6)
+			(end -2.1 1.6)
 			(stroke
 				(width 0.1)
@@
 		)
 		(fp_line
-			(start 1.95 -1.45)
-			(end 1.95 1.45)
+			(start -2.1 1.6)
+			(end 2.1 1.6)
 			(stroke
 				(width 0.1)
@@
 		)
 		(fp_line
-			(start -1.95 1.45)
-			(end -1.95 -1.45)
+			(start -0.4 -1.1)
+			(end 0.4 -1.1)
 			(stroke
 				(width 0.1)
@@
 		)
 		(fp_line
-			(start -1.95 -1.45)
-			(end 1.95 -1.45)
+			(start 0.4 1.1)
+			(end -0.4 1.1)
 			(stroke
 				(width 0.1)
@@
 			(layer "F.Fab")
 		)
-		(fp_circle
-			(center 0 0)
-			(end 1 0)
+		(fp_line
+			(start 2.1 -1.6)
+			(end -2.1 -1.6)
+			(stroke
+				(width 0.1)
+				(type solid)
+			)
+			(layer "F.Fab")
+		)
+		(fp_line
+			(start 2.1 1.6)
+			(end 2.1 -1.6)
+			(stroke
+				(width 0.1)
+				(type solid)
+			)
+			(layer "F.Fab")
+		)
+		(fp_arc
+			(start -0.4 1.1)
+			(mid -1.5 0)
+			(end -0.4 -1.1)
+			(stroke
+				(width 0.1)
+				(type solid)
+			)
+			(layer "F.Fab")
+		)
+		(fp_arc
+			(start 0.4 -1.1)
+			(mid 1.5 0)
+			(end 0.4 1.1)
 			(stroke
 				(width 0.1)
 				(type solid)
 			)
-			(fill no)
 			(layer "F.Fab")
 		)
 		(fp_text user "${REFERENCE}"
-			(at 0 -2.3 0)
+			(at 0 0 0)
 			(layer "F.Fab")
 			(effects
 				(font
-					(size 1 1)
-					(thickness 0.15)
+					(size 0.6 0.6)
+					(thickness 0.09)
 				)
 			)
 		)
-		(pad "1" smd roundrect
-			(at -2.1 0 180)
-			(size 0.8 2)
+		(pad "1" smd rect
+			(at -2.075 -1.075)
+			(size 1.05 0.65)
 			(layers "F.Cu" "F.Mask" "F.Paste")
-			(roundrect_rratio 0.25)
 			(net "GND")
 			(pinfunction "1_1")
 			(pintype "passive")
 		)
-		(pad "2" smd roundrect
-			(at 2.1 0 180)
-			(size 0.8 2)
+		(pad "1" smd rect
+			(at 2.075 -1.075)
+			(size 1.05 0.65)
+			(layers "F.Cu" "F.Mask" "F.Paste")
+			(net "GND")
+			(pinfunction "1_1")
+			(pintype "passive")
+		)
+		(pad "2" smd rect
+			(at -2.075 1.075)
+			(size 1.05 0.65)
+			(layers "F.Cu" "F.Mask" "F.Paste")
+			(net "Net-(R6-Pad1)")
+			(pinfunction "2_2")
+			(pintype "passive")
+		)
+		(pad "2" smd rect
+			(at 2.075 1.075)
+			(size 1.05 0.65)
 			(layers "F.Cu" "F.Mask" "F.Paste")
-			(roundrect_rratio 0.25)
 			(net "Net-(R6-Pad1)")
 			(pinfunction "2_2")
@@
 		)
 		(embedded_fonts no)
-		(model "${KICAD10_3DMODEL_DIR}/Button_Switch_SMD.3dshapes/SW_Push_SPST_NO_Alps_SKRK.step"
+		(model "${KICAD10_3DMODEL_DIR}/Button_Switch_SMD.3dshapes/SW_SPST_PTS810.step"
 			(offset
 				(xyz 0 0 0)
@@
 	)
 	(segment
-		(start 88.7 111.84)
-		(end 88.7 109.775)
+		(start 89.175 110.625)
+		(end 89.175 111.365)
+		(width 0.2)
+		(layer "F.Cu")
+		(net "Net-(R6-Pad1)")
+	)
+	(segment
+		(start 93.325 110.625)
+		(end 89.175 110.625)
+		(width 0.2)
+		(layer "F.Cu")
+		(net "Net-(R6-Pad1)")
+	)
+	(segment
+		(start 89.175 111.365)
+		(end 88.7 111.84)
 		(width 0.2)
 		(layer "F.Cu")
@@
 	)
 	(segment
-		(start 92.532843 115.075)
-		(end 93.539386 115.075)
+		(start 93.140686 115.925)
+		(end 93.539386 115.925)
 		(width 0.2)
 		(layer "F.Cu")
@@
 	)
 	(segment
-		(start 93.539386 115.075)
+		(start 93.75 115.714386)
 		(end 93.75 115.285614)
 		(width 0.2)
@@
 	)
 	(segment
-		(start 93.75 115.285614)
+		(start 93.539386 115.925)
 		(end 93.75 115.714386)
 		(width 0.2)
@@
 	)
 	(segment
-		(start 93.75 115.714386)
-		(end 93.539386 115.925)
+		(start 92.2625 119.4625)
+		(end 92.2625 116.803186)
 		(width 0.2)
 		(layer "F.Cu")
@@
 	(segment
 		(start 92.2625 116.803186)
-		(end 92.2625 119.4625)
+		(end 93.140686 115.925)
 		(width 0.2)
 		(layer "F.Cu")
@@
 	)
 	(segment
-		(start 93.140686 115.925)
-		(end 92.2625 116.803186)
+		(start 93.75 115.285614)
+		(end 93.464386 115)
 		(width 0.2)
 		(layer "F.Cu")
@@
 	)
 	(segment
-		(start 93.539386 115.925)
-		(end 93.140686 115.925)
+		(start 93.464386 115)
+		(end 93 115)
 		(width 0.2)
 		(layer "F.Cu")
