File: _restore_backup_2026-08-06T16-08-01-557/rp-2040 devboard.kicad_pcb (KiCad board)
At the start: 2 copper layers, 20.7 x 51.8 mm, 37 parts, among them J1 USB_C_Receptacle_USB2.0_16P, J2 Conn_01x20, J3 Conn_01x20, J4 Conn_01x03, SW1 SW_Push, U1 RP2040, U2 APS1604M-3SQRx-ZR, U4 MCP1700x-330xxTT, Y1 Crystal_GND24

Commit message: changed PCB and Readme
Parts:
- removed D1, D2: LED, LED_SMD:LED_0402_1005Metric
- removed G***: LOGO, LOGO
- removed R8, R9: 1K, Resistor_SMD:R_0402_1005Metric
Connections:
- U1 pad 37: GPIO25 -> unconnected-(U1-GPIO25-Pad37)
Routing:
- net GPIO25: track 9.93 -> 0.00 mm, vias 2 -> 0
- net VBUS: track 27.0 -> 23.6 mm
- net Net-(D1-A): track 1.47 -> 0.00 mm
- net Net-(D2-A): track 1.17 -> 0.00 mm
- net GND: track 12.5 -> 13.6 mm
Other:
- board text removed: "Made by Ahad Khatri"
