File: _restore_backup_2026-08-06T16-08-01-557/rp-2040 devboard.kicad_sch (KiCad schematic)
At the start: 33 parts, among them J1 USB_C_Receptacle_USB2.0_16P, J2 Conn_01x20, J3 Conn_01x20, J4 Conn_01x03, SW1 SW_Push, U1 RP2040, U2 APS1604M-3SQRx-ZR, U4 MCP1700x-330xxTT, Y1 Crystal_GND24

Commit message: changed PCB and Readme
Parts:
- D1, D2: footprint LED_SMD:LED_0402_1005Metric -> (none)
Changed lines of the file:
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@@
 			)
 		)
-		(property "Footprint" "LED_SMD:LED_0402_1005Metric"
+		(property "Footprint" ""
 			(at 60.96 39.37 0)
 			(hide yes)
@@
 			)
 		)
-		(property "Footprint" "LED_SMD:LED_0402_1005Metric"
+		(property "Footprint" ""
 			(at 48.26 39.37 0)
 			(hide yes)
